Commit message: 调整膨胀半径和仿真惯性参数

File: src/rdk_robot_bringup/urdf/rdk_robot_gazebo.urdf (robot description, URDF)
Before this commit: robot rdk_robot, 7 links, 6 joints
Links:
- link base_link: mass 2.0 -> 0.55
- link front_caster: mass 0.05 -> 0.02; geometry collision sphere radius=0.018; visual sphere radius=0.018
- link imu_link: mass 0.02 -> 0.01
- link laser_frame: mass 0.1 -> 0.08
- link left_wheel: mass 0.15 -> 0.06
- link right_wheel: mass 0.15 -> 0.06
Joints:
- joint caster_joint: origin xyz=0.1 0 -0.016 rpy=0 0 0 -> xyz=0.1 0 -0.022 rpy=0 0 0
